File: PCB_Designs/SMD_QFN_Touch/QFN_Touch.kicad_sch (KiCad schematic)
At the start: 15 parts, among them J1 USB-AM-S-X-X-TH, U1 ATtiny85-20M, Y1 12MHz

Commit message: Update QFN touch pad PCB design files and README
- Modified KiCad project and schematic files for SMD QFN touch pad using TTP223 IC
- Deleted unnecessary auto-saved and lock files from the project directory
- Added images of the QFN Touch PCB design
- Updated README to include details on the 4-layer PCB design
Parts:
- D1, D2: footprint LED_SMD:LED_0201_0603Metric_Pad0.64x0.40mm_HandSolder -> Library:LED_Kingbright_APA1606_1.6x0.6mm_Horizontal_NEW
Changed lines of the file:
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@@
 			)
 		)
-		(property "Footprint" "LED_SMD:LED_0201_0603Metric_Pad0.64x0.40mm_HandSolder"
+		(property "Footprint" "Library:LED_Kingbright_APA1606_1.6x0.6mm_Horizontal_NEW"
 			(at 54.61 71.12 0)
 			(effects
@@
 			)
 		)
-		(property "Footprint" "LED_SMD:LED_0201_0603Metric_Pad0.64x0.40mm_HandSolder"
+		(property "Footprint" "Library:LED_Kingbright_APA1606_1.6x0.6mm_Horizontal_NEW"
 			(at 109.22 109.22 0)
 			(effects
